File: power.kicad_sch (KiCad schematic)
At the start: 33 parts, among them Q4 CSD17575Q3, Q5 CSD17312Q5, U10 DS4432U+, U16 LM27402, U9 INA260

Commit message: all the footprints are in?
Parts:
- Q5: footprint (none) -> blockaxe:DQH8
Connections:
- net PAD: now also U16.17 (PAD); no longer U16.EP (PAD)
Changed lines of the file:
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@@
       (effects (font (size 1.27 1.27)) (justify left))
     )
-    (property "Footprint" "" (at 175.26 45.085 0)
+    (property "Footprint" "blockaxe:DQH8" (at 175.26 45.085 0)
       (effects (font (size 1.27 1.27)) hide)
     )
@@
     )
   )
-  (symbol (lib_name "LM27402SQ_NOPB_1") (lib_id "blockaxe:LM27402SQ_NOPB") (at 134.62 55.88 0) (unit 1)
+  (symbol (lib_id "blockaxe:LM27402SQ_NOPB") (at 134.62 55.88 0) (unit 1)
     (in_bom yes) (on_board yes) (dnp no)
     (property "Reference" "U16" (at 120.015 41.91 0)
@@
       (effects (font (size 1.27 1.27) italic) hide)
     )
-    (property "Datasheet" "https://www.ti.com/lit/ds/symlink/lm27402.pdf" (at 165.1 39.37 0)
+    (property "Datasheet" "LM27402SQ/NOPB" (at 165.1 39.37 0)
       (effects (font (size 1.27 1.27) italic) hide)
     )
@@
     (pin "8")
     (pin "9")
-    (pin "EP")
+    (pin "17")
     (instances
       (project "blockaxe1"

Commit message: routed the buck reg. started placing board
Parts:
- removed R22: 56.2k, Resistor_SMD:R_0402_1005Metric, symbol Device:R_US
- C55: footprint Capacitor_SMD:C_0201_0603Metric -> Capacitor_SMD:C_0603_1608Metric
Connections:
- net PGOOD: now also U16.8 (PGOOD)
Other:
- moved on the sheet: C57, C58, R24

Commit message: more placing and routing
Connections:
- net SW: now reaches C54.2, L2.1, Q4.1, Q4.2, Q4.3 (S), Q5.5 (D), R26.1, U16.12 (SW)
Other:
- moved on the sheet: C54
Changed lines of the file:
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@@
   (junction (at 74.295 22.225) (diameter 0) (color 0 0 0 0)
   )
+  (junction (at 104.14 37.465) (diameter 0) (color 0 0 0 0)
+  )
   (junction (at 222.885 88.265) (diameter 0) (color 0 0 0 0)
   )
   (junction (at 85.09 88.265) (diameter 0) (color 0 0 0 0)
   )
-  (junction (at 160.02 37.465) (diameter 0) (color 0 0 0 0)
-  )
   (junction (at 154.94 67.945) (diameter 0) (color 0 0 0 0)
   )
@@
   )
   (junction (at 222.885 62.865) (diameter 0) (color 0 0 0 0)
-  )
-  (junction (at 106.045 37.465) (diameter 0) (color 0 0 0 0)
   )
   (junction (at 134.62 88.265) (diameter 0) (color 0 0 0 0)
@@
     (stroke (width 0) (type default))
   )
-  (wire (pts (xy 116.84 37.465) (xy 160.02 37.465))
-    (stroke (width 0) (type default))
-  )
   (wire (pts (xy 134.62 27.305) (xy 81.28 27.305))
     (stroke (width 0) (type default))
   )
-  (wire (pts (xy 106.045 46.99) (xy 106.045 37.465))
+  (wire (pts (xy 104.14 46.99) (xy 104.14 37.465))
     (stroke (width 0) (type default))
   )
@@
     (stroke (width 0) (type default))
   )
-  (wire (pts (xy 106.045 37.465) (xy 109.22 37.465))
-    (stroke (width 0) (type default))
-  )
   (wire (pts (xy 74.295 43.815) (xy 74.295 53.34))
     (stroke (width 0) (type default))
   )
+  (wire (pts (xy 104.14 37.465) (xy 106.68 37.465))
+    (stroke (width 0) (type default))
+  )
   (wire (pts (xy 63.627 142.494) (xy 61.722 142.494))
     (stroke (width 0) (type default))
@@
     (stroke (width 0) (type default))
   )
-  (wire (pts (xy 85.09 37.465) (xy 106.045 37.465))
+  (wire (pts (xy 85.09 37.465) (xy 104.14 37.465))
     (stroke (width 0) (type default))
   )
@@
     (stroke (width 0) (type default))
   )
+  (wire (pts (xy 114.3 37.465) (xy 122.555 37.465))
+    (stroke (width 0) (type default))
+  )
   (wire (pts (xy 215.265 127.635) (xy 222.885 127.635))
     (stroke (width 0) (type default))
@@
     (stroke (width 0) (type default))
   )
-  (wire (pts (xy 116.84 46.99) (xy 106.045 46.99))
+  (wire (pts (xy 116.84 46.99) (xy 104.14 46.99))
     (stroke (width 0) (type default))
   )
@@
     (effects (font (size 1.27 1.27)) (justify left bottom))
   )
+  (label "SW" (at 165.735 37.465 180) (fields_autoplaced)
+    (effects (font (size 1.27 1.27)) (justify right bottom))
+  )
   (label "SCL" (at 87.757 145.034 0) (fields_autoplaced)
     (effects (font (size 1.27 1.27)) (justify left bottom))
+  )
+  (label "SW" (at 122.555 37.465 180) (fields_autoplaced)
+    (effects (font (size 1.27 1.27)) (justify right bottom))
   )
   (global_label "GND" (shape input) (at 260.985 88.265 0) (fields_autoplaced)
@@
     )
   )
-  (symbol (lib_id "Device:C") (at 113.03 37.465 90) (unit 1)
+  (symbol (lib_id "Device:C") (at 110.49 37.465 90) (unit 1)
     (in_bom yes) (on_board yes) (dnp no) (fields_autoplaced)
-    (property "Reference" "C54" (at 113.03 30.48 90)
+    (property "Reference" "C54" (at 110.49 30.48 90)
       (effects (font (size 1.27 1.27)))
     )
-    (property "Value" "220nF" (at 113.03 33.02 90)
+    (property "Value" "220nF" (at 110.49 33.02 90)
       (effects (font (size 1.27 1.27)))
     )
-    (property "Footprint" "Capacitor_SMD:C_0603_1608Metric" (at 116.84 36.4998 0)
-      (effects (font (size 1.27 1.27)) hide)
-    )
-    (property "Datasheet" "~" (at 113.03 37.465 0)
-      (effects (font (size 1.27 1.27)) hide)
-    )
+    (property "Footprint" "Capacitor_SMD:C_0603_1608Metric" (at 114.3 36.4998 0)
+      (effects (font (size 1.27 1.27)) hide)
+    )
+    (property "Datasheet" "~" (at 110.49 37.465 0)
+      (effects (font (size 1.27 1.27)) hide)
+    )

Commit message: more routing. switched to RA buttons, moved the buck closer to the barrel
Parts:
- removed R6: 10k, Resistor_SMD:R_0402_1005Metric, symbol Device:R_US
Changed lines of the file:
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@@
   (junction (at 176.53 37.465) (diameter 0) (color 0 0 0 0)
-  )
-  (junction (at 141.732 128.524) (diameter 0) (color 0 0 0 0)
   )
   (junction (at 247.65 37.465) (diameter 0) (color 0 0 0 0)
@@
     (stroke (width 0) (type default))
   )
-  (wire (pts (xy 116.84 54.61) (xy 106.68 54.61))
+  (wire (pts (xy 98.425 54.61) (xy 116.84 54.61))
     (stroke (width 0) (type default))
   )
@@
     (stroke (width 0) (type default))
   )
-  (wire (pts (xy 141.732 125.984) (xy 141.732 128.524))
-    (stroke (width 0) (type default))
-  )
   (wire (pts (xy 165.735 78.74) (xy 154.94 78.74))
     (stroke (width 0) (type default))
@@
     (stroke (width 0) (type default))
   )
-  (wire (pts (xy 130.302 128.524) (xy 141.732 128.524))
-    (stroke (width 0) (type default))
-  )
   (wire (pts (xy 83.947 147.574) (xy 96.012 147.574))
     (stroke (width 0) (type default))
@@
     (stroke (width 0) (type default))
   )
-  (wire (pts (xy 141.732 128.524) (xy 152.527 128.524))
-    (stroke (width 0) (type default))
-  )
   (wire (pts (xy 160.02 52.07) (xy 160.02 37.465))
     (stroke (width 0) (type default))
   )
   (wire (pts (xy 134.62 88.265) (xy 222.885 88.265))
-    (stroke (width 0) (type default))
-  )
-  (wire (pts (xy 141.732 112.014) (xy 141.732 118.364))
     (stroke (width 0) (type default))
   )
@@
     (effects (font (size 1.27 1.27)) (justify left bottom))
   )
-  (label "PGOOD" (at 132.842 128.524 0) (fields_autoplaced)
-    (effects (font (size 1.27 1.27)) (justify left bottom))
-  )
   (label "GND" (at 229.235 149.225 0) (fields_autoplaced)
     (effects (font (size 1.27 1.27)) (justify left bottom))
@@
   )
   (label "GND" (at 172.72 55.88 0) (fields_autoplaced)
-    (effects (font (size 1.27 1.27)) (justify left bottom))
-  )
-  (label "3V3" (at 141.732 115.824 0) (fields_autoplaced)
     (effects (font (size 1.27 1.27)) (justify left bottom))
   )
@@
     (effects (font (size 1.27 1.27)) (justify right))
   )
-  (hierarchical_label "PGOOD" (shape output) (at 152.527 128.524 0) (fields_autoplaced)
-    (effects (font (size 1.27 1.27)) (justify left))
+  (hierarchical_label "PGOOD" (shape output) (at 98.425 54.61 180) (fields_autoplaced)
+    (effects (font (size 1.27 1.27)) (justify right))
   )
   (hierarchical_label "3V3" (shape input) (at 73.787 128.524 0) (fields_autoplaced)
@@
         )
       )
-      (project "power"
-        (path "/d3eaf28f-d55a-4d77-ac4e-fd16c6984c1a"
-          (reference "R4") (unit 1)
-        )
-      )
-      (project "bitaxeUltra"
-        (path "/e63e39d7-6ac0-4ffd-8aa3-1841a4541b55/8ec0a9c6-2b78-44ef-a83d-9047d2828409"
-          (reference "R4") (unit 1)
-        )
-      )
-    )
-  )
-  (symbol (lib_id "Device:R_US") (at 141.732 122.174 0) (unit 1)
-    (in_bom yes) (on_board yes) (dnp no) (fields_autoplaced)
-    (property "Reference" "R6" (at 144.272 120.9039 0)
-      (effects (font (size 1.27 1.27)) (justify left))
-    )
-    (property "Value" "10k" (at 144.272 123.4439 0)
-      (effects (font (size 1.27 1.27)) (justify left))
-    )
-    (property "Footprint" "Resistor_SMD:R_0402_1005Metric" (at 142.748 122.428 90)
-      (effects (font (size 1.27 1.27)) hide)
-    )
-    (property "Datasheet" "~" (at 141.732 122.174 0)
-      (effects (font (size 1.27 1.27)) hide)
-    )
-    (property "DK" "311-10KJRCT-ND" (at 141.732 122.174 0)
-      (effects (font (size 1.27 1.27)) hide)
-    )
-    (property "PARTNO" "RC0402JR-0710KL" (at 141.732 122.174 0)
-      (effects (font (size 1.27 1.27)) hide)
-    )
-    (pin "1")
-    (pin "2")
-    (instances
-      (project "blockaxe1"
-        (path "/a166cb37-4e3a-4be5-b2da-277a3281a4de/b1ac536e-1817-4330-9049-6608155edca8"
-          (reference "R6") (unit 1)
-        )
-      )

Commit message: added gerbers and BOM
Parts:
- C53: DK (none) -> 1276-1066-1-ND; PARTNO (none) -> CL21B105KAFNNNE
- C54: value 220nF -> 0.22uF; DK (none) -> 490-3290-1-ND; PARTNO (none) -> GRM188R71E224KA88D
- C55: footprint Capacitor_SMD:C_0603_1608Metric -> Capacitor_SMD:C_0805_2012Metric; DK (none) -> 1276-1066-1-ND; PARTNO (none) -> CL21B105KAFNNNE
- C56: value 27nF -> 0.027uF; DK (none) -> 1292-1200-1-ND; PARTNO (none) -> 0402B273K250CT
- C57: value 1nF -> 0.001uF; DK (none) -> 478-KGM21NR71H102KTCT-ND; PARTNO (none) -> KGM21NR71H102KT
- C58: DK (none) -> 311-1110-1-ND; PARTNO (none) -> CC0805JRNPO9BN820
- C59: DK (none) -> 311-1024-1-ND; PARTNO (none) -> CC0402JRNPO9BN101
- C60: DK (none) -> 1276-1164-1-ND; PARTNO (none) -> CL21C221JBANNNC
- C62: value 220nF -> 0.22uF; footprint Capacitor_SMD:C_0402_1005Metric -> Capacitor_SMD:C_0603_1608Metric; DK (none) -> 490-3290-1-ND; PARTNO (none) -> GRM188R71E224KA88D
- R21: DK (none) -> RMCF0402FT2R21CT-ND; PARTNO (none) -> RMCF0402FT2R21
- R23: DK (none) -> YAG2958CT-ND; PARTNO (none) -> RC0402FR-0711K8L
- R24: DK (none) -> YAG3195CT-ND; PARTNO (none) -> RC0402FR-075K23L
- R25, R27: DK (none) -> YAG3208CT-ND; PARTNO (none) -> RC0402FR-07665RL
- R26: DK (none) -> 311-2.67KLRCT-ND; PARTNO (none) -> RC0402FR-072K67L
- R28: DK (none) -> P20.0KLCT-ND; PARTNO (none) -> ERJ-2RKF2002X
- R29: DK (none) -> YAG3162CT-ND; PARTNO (none) -> RC0402FR-07442RL
- R30: DK (none) -> 311-120KLRCT-ND; PARTNO (none) -> RC0402FR-07120KL
Changed lines of the file:
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@@
+      (effects (font (size 1.27 1.27)) hide)
+    )
+    (property "DK" "YAG3208CT-ND" (at 212.725 53.975 0)
+      (effects (font (size 1.27 1.27)) hide)
+    )
+    (property "PARTNO" "RC0402FR-07665RL" (at 212.725 53.975 0)
       (effects (font (size 1.27 1.27)) hide)
     )
@@
     )
     (property "Datasheet" "~" (at 198.755 53.975 0)
+      (effects (font (size 1.27 1.27)) hide)
+    )
+    (property "DK" "YAG3208CT-ND" (at 198.755 53.975 0)
+      (effects (font (size 1.27 1.27)) hide)
+    )
+    (property "PARTNO" "RC0402FR-07665RL" (at 198.755 53.975 0)
       (effects (font (size 1.27 1.27)) hide)
     )
@@
       (effects (font (size 1.27 1.27)) hide)
     )
+    (property "DK" "P20.0KLCT-ND" (at 222.885 48.895 0)
+      (effects (font (size 1.27 1.27)) hide)
+    )
+    (property "PARTNO" "ERJ-2RKF2002X" (at 222.885 48.895 0)
+      (effects (font (size 1.27 1.27)) hide)
+    )
     (pin "1")
     (pin "2")
@@
       (effects (font (size 1.27 1.27)))
     )
-    (property "Value" "220nF" (at 110.49 33.02 90)
+    (property "Value" "0.22uF" (at 110.49 33.02 90)
       (effects (font (size 1.27 1.27)))
     )
@@
     )
     (property "Datasheet" "~" (at 110.49 37.465 0)
+      (effects (font (size 1.27 1.27)) hide)
+    )
+    (property "DK" "490-3290-1-ND" (at 110.49 37.465 0)
+      (effects (font (size 1.27 1.27)) hide)
+    )
+    (property "PARTNO" "GRM188R71E224KA88D" (at 110.49 37.465 0)
       (effects (font (size 1.27 1.27)) hide)
     )
@@
       (effects (font (size 1.27 1.27)) hide)
     )
+    (property "DK" "YAG2958CT-ND" (at 109.855 75.565 0)
+      (effects (font (size 1.27 1.27)) hide)
+    )
+    (property "PARTNO" "RC0402FR-0711K8L" (at 109.855 75.565 0)
+      (effects (font (size 1.27 1.27)) hide)
+    )
     (pin "1")
     (pin "2")
@@
       (effects (font (size 1.27 1.27)) (justify left))
     )
-    (property "Footprint" "Capacitor_SMD:C_0603_1608Metric" (at 86.0552 79.375 0)
+    (property "Footprint" "Capacitor_SMD:C_0805_2012Metric" (at 86.0552 79.375 0)
       (effects (font (size 1.27 1.27)) hide)
     )
@@
       (effects (font (size 1.27 1.27)) hide)
     )
+    (property "DK" "1276-1066-1-ND" (at 85.09 75.565 0)
+      (effects (font (size 1.27 1.27)) hide)
+    )
+    (property "PARTNO" "CL21B105KAFNNNE" (at 85.09 75.565 0)
+      (effects (font (size 1.27 1.27)) hide)
+    )
     (pin "1")
     (pin "2")
@@
     )
     (property "Datasheet" "~" (at 177.165 67.945 0)
+      (effects (font (size 1.27 1.27)) hide)
+    )
+    (property "DK" "YAG3195CT-ND" (at 177.165 67.945 0)
+      (effects (font (size 1.27 1.27)) hide)
+    )
+    (property "PARTNO" "RC0402FR-075K23L" (at 177.165 67.945 0)
       (effects (font (size 1.27 1.27)) hide)
     )
@@
       (effects (font (size 1.27 1.27)) hide)
     )
+    (property "DK" "311-120KLRCT-ND" (at 222.885 79.375 0)
+      (effects (font (size 1.27 1.27)) hide)
+    )
+    (property "PARTNO" "RC0402FR-07120KL" (at 222.885 79.375 0)
+      (effects (font (size 1.27 1.27)) hide)
+    )
     (pin "1")
     (pin "2")
@@
     )
     (property "Datasheet" "~" (at 192.405 46.355 0)
+      (effects (font (size 1.27 1.27)) hide)
+    )
+    (property "DK" "311-2.67KLRCT-ND" (at 192.405 46.355 0)
+      (effects (font (size 1.27 1.27)) hide)
+    )
+    (property "PARTNO" "RC0402FR-072K67L" (at 192.405 46.355 0)
       (effects (font (size 1.27 1.27)) hide)
     )
@@
       (effects (font (size 1.27 1.27)))
     )
-    (property "Value" "1nF" (at 166.37 66.675 90)
+    (property "Value" "0.001uF" (at 166.37 66.675 90)
       (effects (font (size 1.27 1.27)))
     )
@@
       (effects (font (size 1.27 1.27)) hide)
     )
+    (property "DK" "478-KGM21NR71H102KTCT-ND" (at 162.56 67.945 0)
+      (effects (font (size 1.27 1.27)) hide)
+    )
+    (property "PARTNO" "KGM21NR71H102KT" (at 162.56 67.945 0)
+      (effects (font (size 1.27 1.27)) hide)
+    )
     (pin "1")
     (pin "2")
@@
       (effects (font (size 1.27 1.27)))
     )
-    (property "Value" "220nF" (at 205.74 42.545 90)
-      (effects (font (size 1.27 1.27)))
-    )
-    (property "Footprint" "Capacitor_SMD:C_0402_1005Metric" (at 209.55 45.3898 0)
+    (property "Value" "0.22uF" (at 205.74 42.545 90)
+      (effects (font (size 1.27 1.27)))
+    )
+    (property "Footprint" "Capacitor_SMD:C_0603_1608Metric" (at 209.55 45.3898 0)
       (effects (font (size 1.27 1.27)) hide)
     )
     (property "Datasheet" "~" (at 205.74 46.355 0)
+      (effects (font (size 1.27 1.27)) hide)
+    )
+    (property "DK" "490-3290-1-ND" (at 205.74 46.355 0)
+      (effects (font (size 1.27 1.27)) hide)
+    )
+    (property "PARTNO" "GRM188R71E224KA88D" (at 205.74 46.355 0)
       (effects (font (size 1.27 1.27)) hide)
     )
@@
       (effects (font (size 1.27 1.27)) hide)
     )
+    (property "DK" "311-1024-1-ND" (at 205.74 61.595 0)
+      (effects (font (size 1.27 1.27)) hide)
+    )
+    (property "PARTNO" "CC0402JRNPO9BN101" (at 205.74 61.595 0)
+      (effects (font (size 1.27 1.27)) hide)
+    )
     (pin "1")
     (pin "2")
@@
       (effects (font (size 1.27 1.27)) hide)
     )
+    (property "DK" "RMCF0402FT2R21CT-ND" (at 74.295 34.925 0)
+      (effects (font (size 1.27 1.27)) hide)
+    )
+    (property "PARTNO" "RMCF0402FT2R21" (at 74.295 34.925 0)
+      (effects (font (size 1.27 1.27)) hide)
+    )
     (pin "1")
     (pin "2")
@@
       (effects (font (size 1.27 1.27)) hide)
     )
+    (property "DK" "YAG3162CT-ND" (at 234.315 56.515 0)
+      (effects (font (size 1.27 1.27)) hide)
+    )
+    (property "PARTNO" "RC0402FR-07442RL" (at 234.315 56.515 0)
+      (effects (font (size 1.27 1.27)) hide)
+    )
     (pin "1")
     (pin "2")
@@
       (effects (font (size 1.27 1.27)) hide)
     )
+    (property "DK" "1276-1066-1-ND" (at 74.295 57.15 0)
+      (effects (font (size 1.27 1.27)) hide)
+    )
+    (property "PARTNO" "CL21B105KAFNNNE" (at 74.295 57.15 0)
+      (effects (font (size 1.27 1.27)) hide)
+    )
     (pin "1")
     (pin "2")
@@
       (effects (font (size 1.27 1.27)) (justify left))
     )
-    (property "Value" "27nF" (at 101.6 76.835 0)
+    (property "Value" "0.027uF" (at 101.6 76.835 0)
       (effects (font (size 1.27 1.27)) (justify left))
     )
@@
     )
     (property "Datasheet" "~" (at 98.425 75.565 0)
+      (effects (font (size 1.27 1.27)) hide)
+    )
+    (property "DK" "1292-1200-1-ND" (at 98.425 75.565 0)
+      (effects (font (size 1.27 1.27)) hide)
+    )
+    (property "PARTNO" "0402B273K250CT" (at 98.425 75.565 0)
       (effects (font (size 1.27 1.27)) hide)
     )
@@
       (effects (font (size 1.27 1.27)) hide)
     )
+    (property "DK" "1276-1164-1-ND" (at 234.315 43.815 0)
+      (effects (font (size 1.27 1.27)) hide)
+    )
+    (property "PARTNO" "CL21C221JBANNNC" (at 234.315 43.815 0)
+      (effects (font (size 1.27 1.27)) hide)
+    )
     (pin "1")
     (pin "2")
@@
       (effects (font (size 1.27 1.27)) hide)
     )
+    (property "DK" "311-1110-1-ND" (at 169.545 78.74 0)
+      (effects (font (size 1.27 1.27)) hide)
+    )
+    (property "PARTNO" "CC0805JRNPO9BN820" (at 169.545 78.74 0)
+      (effects (font (size 1.27 1.27)) hide)
+    )
