File: power.kicad_sch (KiCad schematic)
At the start: 44 parts, among them U10 TPS82130, U2 TPS546D24SRVFR, U7 TPS82130

Commit message: migrated over the 1103x accessory voltage regulators. started rough parts placement
Parts:
- removed C1, C8: 10uF, Capacitor_SMD:C_0603_1608Metric, symbol Device:C_Small
- removed C12, C29: 3.3nF, Capacitor_SMD:C_0402_1005Metric, symbol Device:C_Small
- removed C30, C31: 22uF, Capacitor_SMD:C_1206_3216Metric, symbol Device:C_Small
- removed R10: 536k, Resistor_SMD:R_0402_1005Metric, symbol Device:R_Small_US
- removed R11, R13: 100k, Resistor_SMD:R_0402_1005Metric, symbol Device:R_Small_US
- removed R12: 309k, Resistor_SMD:R_0402_1005Metric, symbol Device:R_Small_US
- removed TP15: 5V, bitaxe:TestPoint_Pad_D1.0mm, symbol Connector:TestPoint
- removed TP9: 3V3, bitaxe:TestPoint_Pad_D1.0mm, symbol Connector:TestPoint
- removed U10, U7: TPS82130, bitaxe:Texas_SIL0008D_MicroSiP-8-1EP_2.8x3mm_P0.65mm_EP1.1x1.9mm_ThermalVias, symbol bitaxe:TPS82130
- added C49, C50: 10uF, Capacitor_SMD:C_1210_3225Metric, symbol Device:C_Small
- added C51, C52, C55, C56: 0.1uF, Capacitor_SMD:C_0402_1005Metric, symbol Device:C_Small
- added C53, C54: 33nF, Capacitor_SMD:C_0603_1608Metric, symbol Device:C_Small
- added C65, C66: 22uF, Capacitor_SMD:C_0805_2012Metric, symbol Device:C_Small
- added FB1, FB2: FerriteBead, Inductor_SMD:L_1206_3216Metric, symbol Device:FerriteBead
- added L2, L3: 1.5uH, bitaxe:IND-SMD_L2.0-W1.6, symbol Device:L_Small
- added R15, R28: 15k, Resistor_SMD:R_0402_1005Metric, symbol Device:R_Small_US
- added R25: 10k, Resistor_SMD:R_0402_1005Metric, symbol Device:R_Small_US
- added R27: 47k, Resistor_SMD:R_0402_1005Metric, symbol Device:R_Small_US
- added R29: 27k, Resistor_SMD:R_0402_1005Metric, symbol Device:R_Small_US
- added R30: 5.1k, Resistor_SMD:R_0402_1005Metric, symbol Device:R_Small_US
- added TP61: GND, bitaxe:TestPoint_Pad_D1.0mm, symbol Connector:TestPoint
- added TP62: 3V3, bitaxe:TestPoint_Pad_D1.0mm, symbol Connector:TestPoint
- added TP63: 5V, bitaxe:TestPoint_Pad_D1.0mm, symbol Connector:TestPoint
- added U13, U14: TPS62933DRLR, bitaxe:SOT-583-8_L2.1-W1.2-P0.50-LS1.6-BR, symbol bitaxe:TPS62933DRLR
- added U15, U16, U17: STHW4-DU-HN050206, bitaxe:PAD-SMD_L5.0-W2.0_STHW4-DU-HN050206, symbol bitaxe:STHW4-DU-HN050206
Connections:
- net 12V: now also FB1.1, FB2.1
- net 3V3: now also C65.2, L2.2, R27.2, TP62.1
- net 5V: now also C66.2, L3.2, R29.2, TP63.1
- net GND: now also C49.1, C50.1, C51.2, C52.2, C53.1, C54.1, C65.1, C66.1, R15.1, R25.1, R28.1, R30.1, TP61.1, U13.4 (GND), U14.4 (GND), U15.1, U16.1, U17.1
- new net: C53.2, U13.7 (SS)
- new net: C56.2, L3.1, U14.5 (SW)
- new net: C55.1, U13.6 (BST)
- new net: C55.2, L2.1, U13.5 (SW)
- new net: C49.2, C51.1, FB1.2, U13.3 (VIN)
- new net: R25.2, U14.1 (RT)
- new net: C50.2, C52.1, FB2.2, U14.3 (VIN)
- new net: C54.2, U14.7 (SS)
- new net: R15.2, U13.1 (RT)
- new net: R27.1, R28.2, U13.8 (FB)
- new net: C56.1, U14.6 (BST)
- new net: R29.1, R30.2, U14.8 (FB)
Other:
- note added: "3.3V Regulator"
- note added: "5V Regulator"
- note added: "VR Thermal Busbar"

Commit message: changed inductor to Bourns SRP1245A-1R2M as the coilcraft was out of stock everywhere.
Parts:
- C10, C9: LCSC (none) -> C29936
- C11: LCSC (none) -> C23733
- C13: LCSC (none) -> C1538
- C14: LCSC (none) -> C1531
- C17: LCSC (none) -> C46653
- C18: LCSC (none) -> C1546
- C2, C3, C4, C5, C6: LCSC (none) -> C12891
- C20: LCSC (none) -> C96123
- C21, C22, C23, C24: LCSC (none) -> C15008
- L1: footprint bitaxe:XAL1060122MEC -> bitaxe:SRP1245A-180M_BRN; DK 2457-XAL1060-122MEC-ND -> 118-SRP1245A-1R2MCT-ND; LCSC (none) -> C3224581; PARTNO XAL1060-122MEC -> SRP1245A-180M_BRN
- R3: LCSC (none) -> C25744
- R5: LCSC (none) -> C25077
- R6: LCSC (none) -> C253344
- R7, R8: LCSC (none) -> C25120
- U2: LCSC (none) -> C20345977
