File: blockaxe1.kicad_sch (KiCad schematic)
At the start: 16 parts, among them J5 PJ-002B

Commit message: switched barrel plug for #8. touched up schematic, DRC, generated BOM, generated Gerbers
Parts:
- J5: value PJ-002B -> EJ503A; footprint blockaxe:CUI_PJ-002B -> blockaxe:MPD_EJ503A; DK CP-002B-ND -> EJ503A-ND; PARTNO PJ-002B -> EJ503A
Changed lines of the file:
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@@
   (title_block
     (title "blockaxe1")
-    (date "2023-11-15")
-    (rev "1")
+    (date "2024-02-21")
+    (rev "2")
   )
   (junction (at 34.925 167.64) (diameter 0) (color 0 0 0 0)
@@
       (effects (font (size 1.27 1.27)))
     )
-    (property "Value" "PJ-002B" (at 129.032 32.512 0)
+    (property "Value" "EJ503A" (at 129.032 32.512 0)
       (effects (font (size 1.27 1.27)))
     )
-    (property "Footprint" "blockaxe:CUI_PJ-002B" (at 130.302 39.878 0)
-      (effects (font (size 1.27 1.27)) hide)
-    )
-    (property "Datasheet" "~" (at 130.302 39.878 0)
-      (effects (font (size 1.27 1.27)) hide)
-    )
-    (property "DK" "CP-002B-ND" (at 129.032 38.862 0)
-      (effects (font (size 1.27 1.27)) hide)
-    )
-    (property "PARTNO" "PJ-002B" (at 129.032 38.862 0)
+    (property "Footprint" "blockaxe:MPD_EJ503A" (at 130.302 39.878 0)
+      (effects (font (size 1.27 1.27)) hide)
+    )
+    (property "Datasheet" "https://www.memoryprotectiondevices.com/datasheets/EJ503A-datasheet.pdf" (at 130.302 39.878 0)
+      (effects (font (size 1.27 1.27)) hide)
+    )
+    (property "DK" "EJ503A-ND" (at 129.032 38.862 0)
+      (effects (font (size 1.27 1.27)) hide)
+    )
+    (property "PARTNO" "EJ503A" (at 129.032 38.862 0)
       (effects (font (size 1.27 1.27)) hide)
     )
@@
         (path "/e63e39d7-6ac0-4ffd-8aa3-1841a4541b55"
           (reference "FID6") (unit 1)
-        )
-      )
-    )
-  )
-  (symbol (lib_id "blockaxe:LOGO") (at 202.565 173.99 0) (unit 1)
-    (in_bom yes) (on_board yes) (dnp no) (fields_autoplaced)
-    (property "Reference" "#G1" (at 202.565 166.3658 0)
-      (effects (font (size 1.27 1.27)) hide)
-    )
-    (property "Value" "LOGO" (at 202.565 181.6142 0)
-      (effects (font (size 1.27 1.27)) hide)
-    )
-    (property "Footprint" "blockaxe:blockaxe_logo" (at 202.565 173.99 0)
-      (effects (font (size 1.27 1.27)) hide)
-    )
-    (property "Datasheet" "" (at 202.565 173.99 0)
-      (effects (font (size 1.27 1.27)) hide)
-    )
-    (instances
-      (project "blockaxe1"
-        (path "/a166cb37-4e3a-4be5-b2da-277a3281a4de"
-          (reference "#G1") (unit 1)
         )
       )
@@
       (effects (font (size 1.27 1.27)) (justify right))
     )
-    (pin "3V3" input (at 154.432 69.215 0)
-      (effects (font (size 1.27 1.27)) (justify right))
-    )
+    (pin "3V3" input (at 154.432 69.342 0)
+      (effects (font (size 1.27 1.27)) (justify right))
+    )
