File: esp32.kicad_sch (KiCad schematic)
At the start: 12 parts, among them J2 TC2030-IDC, J3 Conn_01x04, J4 Conn_01x08, J5 USB_C_Receptacle_USB2.0, SW1 SWITCH-SPST, SW2 SWITCH-SPST, U5 ESP32-S3-WROOM-1

Commit message: updated TPS546D24 strapping values. fixed inductor value and output capacitors. PCB needs updating to add missing strapping footprint.
Changed lines of the file:
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@@
 	(wire
 		(pts
-			(xy 31.75 121.92) (xy 48.26 121.92)
+			(xy 31.75 76.2) (xy 85.09 76.2)
 		)
 		(stroke
@@
 		(pts
 			(xy 60.96 40.64) (xy 66.04 40.64)
-		)
-		(stroke
-			(width 0)
-			(type default)
-		)
-	)
-	(wire
-		(pts
-			(xy 85.09 76.2) (xy 66.04 76.2)
 		)
 		(stroke
@@
 	(label "IO0"
 		(at 144.78 160.02 180)
-		(effects
-			(font
-				(size 1.27 1.27)
-			)
-			(justify right bottom)
-		)
-	)
-	(label "RST_3V3"
-		(at 48.26 121.92 180)
 		(effects
 			(font
@@
 	(hierarchical_label "RST_3V3"
 		(shape output)
-		(at 31.75 121.92 180)
-		(effects
-			(font
+		(at 31.75 76.2 180)
+		(effects
+			(font
