File: asic.kicad_sch (KiCad schematic)
At the start: 76 parts, among them U1 MCP1824T-1202E/OT, U3 MCP1824T-1202E/OT, U4 MCP1824T-1202E/OT, U6 MCP1824T-1202E/OT, U8 SN74AXC4T774, Y2 50MHz

Commit message: fix pinsel connection on ASIC 3
Connections:
- net DOMAIN1: no longer A3.36 (PINSEL)
- net DOMAIN2: now also A3.36 (PINSEL)
Changed lines of the file:
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@@
 		)
 	)
-	(label "GND2"
+	(label "GND3"
 		(at 259.08 171.45 0)
 		(effects

Commit message: part silkscreen cleanup
Parts:
- U1, U3, U4, U6: footprint Package_TO_SOT_SMD:SOT-23-5 -> bitaxe:SOT-23-5
Connections:
- net DOMAIN1 renamed GND2
- net DOMAIN2 renamed GND3
- net DOMAIN3 renamed GND4
Changed lines of the file:
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@@
 	)
 	(junction
-		(at 287.02 132.08)
-		(diameter 0)
-		(color 0 0 0 0)
-	)
-	(junction
 		(at 481.33 347.98)
 		(diameter 0)
@@
 	)
 	(junction
-		(at 287.02 290.83)
-		(diameter 0)
-		(color 0 0 0 0)
-	)
-	(junction
 		(at 265.43 275.59)
 		(diameter 0)
@@
 	)
 	(junction
-		(at 287.02 213.36)
-		(diameter 0)
-		(color 0 0 0 0)
-	)
-	(junction
 		(at 287.02 62.23)
 		(diameter 0)
@@
 	(wire
 		(pts
-			(xy 287.02 132.08) (xy 287.02 134.62)
-		)
-		(stroke
-			(width 0)
-			(type default)
-		)
-	)
-	(wire
-		(pts
 			(xy 270.51 185.42) (xy 270.51 198.12)
 		)
@@
 	(wire
 		(pts
-			(xy 287.02 132.08) (xy 295.91 132.08)
-		)
-		(stroke
-			(width 0)
-			(type default)
-		)
-	)
-	(wire
-		(pts
 			(xy 516.89 339.09) (xy 516.89 347.98)
 		)
@@
 	(wire
 		(pts
-			(xy 287.02 199.39) (xy 287.02 213.36)
+			(xy 287.02 199.39) (xy 287.02 215.9)
 		)
 		(stroke
@@
 	(wire
 		(pts
-			(xy 287.02 213.36) (xy 295.91 213.36)
-		)
-		(stroke
-			(width 0)
-			(type default)
-		)
-	)
-	(wire
-		(pts
 			(xy 309.88 85.09) (xy 306.07 85.09)
 		)
@@
 	(wire
 		(pts
-			(xy 287.02 213.36) (xy 287.02 215.9)
-		)
-		(stroke
-			(width 0)
-			(type default)
-		)
-	)
-	(wire
-		(pts
 			(xy 217.17 355.6) (xy 265.43 355.6)
 		)
@@
 	(wire
 		(pts
-			(xy 287.02 119.38) (xy 287.02 132.08)
+			(xy 287.02 119.38) (xy 287.02 134.62)
 		)
 		(stroke
@@
 	(wire
 		(pts
-			(xy 287.02 276.86) (xy 287.02 290.83)
-		)
-		(stroke
-			(width 0)
-			(type default)
-		)
-	)
-	(wire
-		(pts
-			(xy 287.02 290.83) (xy 287.02 293.37)
+			(xy 287.02 276.86) (xy 287.02 293.37)
 		)
 		(stroke
@@
 	(wire
 		(pts
-			(xy 287.02 290.83) (xy 295.91 290.83)
-		)
-		(stroke
-			(width 0)
-			(type default)
-		)
-	)
-	(wire
-		(pts
 			(xy 168.91 255.27) (xy 172.72 255.27)
 		)
@@
 		)
 	)
-	(hierarchical_label "DOMAIN2"
-		(shape output)
-		(at 295.91 213.36 0)
-		(effects
-			(font
-				(size 1.27 1.27)
-			)
-			(justify left)
-		)
-	)
-	(hierarchical_label "DOMAIN1"
-		(shape output)
-		(at 295.91 290.83 0)
-		(effects
-			(font
-				(size 1.27 1.27)
-			)
-			(justify left)
-		)
-	)
-	(hierarchical_label "DOMAIN3"
-		(shape output)
-		(at 295.91 132.08 0)
-		(effects
-			(font
-				(size 1.27 1.27)
-			)
-			(justify left)
-		)
-	)
 	(hierarchical_label "RX_3V3"
 		(shape input)
@@
 			)
 		)
-		(property "Footprint" "Package_TO_SOT_SMD:SOT-23-5"
+		(property "Footprint" "bitaxe:SOT-23-5"
 			(at 157.48 163.83 0)
 			(effects
@@
 			)
 		)
-		(property "Footprint" "Package_TO_SOT_SMD:SOT-23-5"
+		(property "Footprint" "bitaxe:SOT-23-5"
 			(at 157.48 242.57 0)
 			(effects
@@
 			)
 		)
-		(property "Footprint" "Package_TO_SOT_SMD:SOT-23-5"
+		(property "Footprint" "bitaxe:SOT-23-5"
 			(at 157.48 85.09 0)
 			(effects
@@
 			)
 		)
-		(property "Footprint" "Package_TO_SOT_SMD:SOT-23-5"
+		(property "Footprint" "bitaxe:SOT-23-5"
 			(at 157.48 316.23 0)
 			(effects
