File: BitaxeBonanza.kicad_sch (KiCad schematic)
At the start: 10 parts, among them J1 XT30

Commit message: migrated over the 1103x accessory voltage regulators. started rough parts placement
Parts:
- removed H1, H2, H3, H4: MountingHole_Pad, MountingHole:MountingHole_3.2mm_M3_Pad_Via, symbol Mechanical:MountingHole_Pad
- added H1, H2, H3, H4, H5, H6, H7, H8: MountingHole_Pad, bitaxe:MountingHole_3.2mm_M3, symbol Mechanical:MountingHole
Other:
- note added: "Case Mounts"
- note added: "PCB Mounts"
