File: BitaxeBonanza.kicad_sch (KiCad schematic)
At the start: 14 parts, among them J1 XT30

Commit message: switched display connector to BAP pins and UART instead of I2C. Bridge is now only ASIC serial. Added ESP32 ADC connections to domain midpoints.
Other:
- sheet ASIC ports: added D1, D2, D3; removed none
- sheet Data ports: added D1, D2, D3; removed none
Changed lines of the file:
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@@
+	(wire
+		(pts
+			(xy 162.56 71.12) (xy 162.56 125.73)
+		)
+		(stroke
+			(width 0)
+			(type default)
+		)
+	)
 	(wire
 		(pts
@@
 	(wire
 		(pts
+			(xy 165.1 73.66) (xy 198.12 73.66)
+		)
+		(stroke
+			(width 0)
+			(type default)
+		)
+	)
+	(wire
+		(pts
 			(xy 128.27 109.22) (xy 148.59 109.22)
 		)
@@
 	(wire
 		(pts
+			(xy 165.1 128.27) (xy 165.1 73.66)
+		)
+		(stroke
+			(width 0)
+			(type default)
+		)
+	)
+	(wire
+		(pts
 			(xy 153.67 60.96) (xy 198.12 60.96)
 		)
@@
 	(wire
 		(pts
+			(xy 167.64 76.2) (xy 167.64 130.81)
+		)
+		(stroke
+			(width 0)
+			(type default)
+		)
+	)
+	(wire
+		(pts
+			(xy 198.12 76.2) (xy 167.64 76.2)
+		)
+		(stroke
+			(width 0)
+			(type default)
+		)
+	)
+	(wire
+		(pts
 			(xy 186.69 121.92) (xy 198.12 121.92)
 		)
@@
 	(wire
 		(pts
+			(xy 162.56 125.73) (xy 128.27 125.73)
+		)
+		(stroke
+			(width 0)
+			(type default)
+		)
+	)
+	(wire
+		(pts
 			(xy 102.87 69.85) (xy 96.52 69.85)
 		)
@@
 	(wire
 		(pts
+			(xy 167.64 130.81) (xy 128.27 130.81)
+		)
+		(stroke
+			(width 0)
+			(type default)
+		)
+	)
+	(wire
+		(pts
 			(xy 128.27 66.04) (xy 135.89 66.04)
 		)
@@
 	(wire
 		(pts
+			(xy 128.27 128.27) (xy 165.1 128.27)
+		)
+		(stroke
+			(width 0)
+			(type default)
+		)
+	)
+	(wire
+		(pts
 			(xy 186.69 118.11) (xy 198.12 118.11)
 		)
@@
 		(pts
 			(xy 78.74 124.46) (xy 78.74 44.45)
+		)
+		(stroke
+			(width 0)
+			(type default)
+		)
+	)
+	(wire
+		(pts
+			(xy 198.12 71.12) (xy 162.56 71.12)
 		)
 		(stroke
@@
 			)
 		)
+		(pin "D1" input
+			(at 128.27 125.73 0)
+			(effects
+				(font
+					(size 1.27 1.27)
+				)
+				(justify right)
+			)
+		)
+		(pin "D2" input
+			(at 128.27 128.27 0)
+			(effects
+				(font
+					(size 1.27 1.27)
+				)
+				(justify right)
+			)
+		)
+		(pin "D3" input
+			(at 128.27 130.81 0)
+			(effects
+				(font
+					(size 1.27 1.27)
+				)
+				(justify right)
+			)
+		)
 		(instances
 			(project "bitaxeBonanza"
@@
 			(effects
 				(font
+					(size 1.27 1.27)
+				)
+				(justify left)
+			)
+		)
+		(pin "D1" output
+			(at 198.12 71.12 180)
+			(effects
+				(font
+					(size 1.27 1.27)
+				)
+				(justify left)
+			)
+		)
+		(pin "D2" output
+			(at 198.12 73.66 180)
+			(effects
+				(font
+					(size 1.27 1.27)
+				)
+				(justify left)
+			)
+		)
+		(pin "D3" output
+			(at 198.12 76.2 180)
+			(effects
+				(font

Commit message: adding jlcpcb deets
Parts:
- J1: FT Origin (none) -> Center; FT Rotation Offset (none) -> 180
Changed lines of the file:
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@@
 			)
 		)
-	)
+		(property "FT Origin" "Center"
+			(at 50.8 45.72 0)
+			(hide yes)
+			(effects
+				(font
+					(size 1.27 1.27)
+				)
+			)
+		)
+		(property "FT Rotation Offset" "180"
+			(at 50.8 45.72 0)
+			(hide yes)
+			(effects
+				(font
+					(size 1.27 1.27)
+				)
+			)
+		))
 	(symbol
 		(lib_id "Mechanical:Fiducial")
