File: shifter.kicad_sch (KiCad schematic)
At the start: 11 parts

Commit message: changed inductor to Bourns SRP1245A-1R2M as the coilcraft was out of stock everywhere.
Parts:
- C142: LCSC (none) -> C1523
- D1, D2, D3, D4: value DLLFSD01T-7 -> BAS516; DK DLLFSD01T-7DICT-ND -> (none); LCSC (none) -> C7502722; Manufacturer (none) -> hongjiacheng; PARTNO DLLFSD01T-7 -> BAS516
- R35, R36, R37, R38, R39, R40: LCSC (none) -> C11702
